File: lexus-qs/board/board.kicad_pcb (KiCad board)
At the start: 2 copper layers, 35.6 x 48.3 mm, 6 parts, among them J1 Conn_01x06_Socket, J2 Conn_01x06_Socket, U2 ADG729

Commit message: Got it to production ready!
Parts:
- RV1, RV2: footprint Potentiometer_SMD:Potentiometer_Bourns_3314R-1_Vertical_Hole -> Potentiometer_SMD:Potentiometer_Bourns_3314J_Vertical
- moved RV2 1.72 mm to (171.0, 88.7)
- moved RV1 1.60 mm to (163.5, 88.9)
Routing:
- net Net-(J1-Pin_2): track 0.00 -> 90.4 mm, vias 0 -> 3
- net Net-(A1-D5): track 0.00 -> 41.4 mm
- net Net-(A1-D7): track 0.00 -> 41.0 mm
- net Net-(A1-D6): track 0.00 -> 37.7 mm
- net Net-(J1-Pin_4): track 0.00 -> 33.5 mm
- net Net-(J1-Pin_3): track 0.00 -> 28.1 mm
- net Net-(J1-Pin_6): track 0.00 -> 26.3 mm
- net Net-(J1-Pin_5): track 0.00 -> 25.7 mm
- net Net-(U2-S2A): track 0.00 -> 24.1 mm
- net Net-(U2-S3A): track 0.00 -> 23.8 mm, vias 0 -> 2
- net Net-(A1-VIN): track 61.9 -> 79.8 mm, vias 0 -> 1
- net Net-(A1-A4): track 0.00 -> 12.8 mm, vias 0 -> 1
- net Net-(A1-A5): track 0.00 -> 8.96 mm, vias 0 -> 1
