File: lexus-qs/board/board.kicad_sch (KiCad schematic)
At the start: 6 parts, among them J1 Conn_01x06_Socket, J2 Conn_01x06_Socket, U2 ADG729

Commit message: Got it to production ready!
Parts:
- J1, J2: LCSC (none) -> C265105
- RV1, RV2: footprint Potentiometer_SMD:Potentiometer_Bourns_3314R-1_Vertical_Hole -> Potentiometer_SMD:Potentiometer_Bourns_3314J_Vertical; LCSC (none) -> C36376
- U2: LCSC (none) -> C207556
Connections:
- net at A1.30 (VIN), J1.1 (Pin_1), RV1.1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: now also U2.14 (VDD)
- net at A1.17 (3V3): no longer U2.14 (VDD)

Commit message: Update board for my goofd
Connections:
- net at A1.29 (GND), J1.2 (Pin_2), RV1.3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: now also U2.16 (A0), U2.2 (A1)
- net at A1.23 (A4): now also U2.3 (SDA); no longer U2.1 (SCL)
- net at A1.24 (A5): now also U2.1 (SCL); no longer U2.3 (SDA)
Changed lines of the file:
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@@
+	)
+	(junction
+		(at 86.36 88.9)
+		(diameter 0)
+		(color 0 0 0 0)
 	)
 	(junction
@@
 	)
 	(junction
+		(at 78.74 120.65)
+		(diameter 0)
+		(color 0 0 0 0)
+	)
+	(junction
 		(at 77.47 62.23)
 		(diameter 0)
@@
 	(wire
 		(pts
+			(xy 49.53 107.95) (xy 58.42 107.95)
+		)
+		(stroke
+			(width 0)
+			(type default)
+		)
+	)
+	(wire
+		(pts
 			(xy 63.5 87.63) (xy 63.5 97.79)
 		)
@@
 	(wire
 		(pts
+			(xy 90.17 88.9) (xy 86.36 88.9)
+		)
+		(stroke
+			(width 0)
+			(type default)
+		)
+	)
+	(wire
+		(pts
 			(xy 121.92 62.23) (xy 105.41 62.23)
 		)
@@
 	(wire
 		(pts
-			(xy 62.23 107.95) (xy 49.53 107.95)
-		)
-		(stroke
-			(width 0)
-			(type default)
-		)
-	)
-	(wire
-		(pts
 			(xy 68.58 62.23) (xy 68.58 71.12)
 		)
@@
 	(wire
 		(pts
+			(xy 78.74 88.9) (xy 78.74 120.65)
+		)
+		(stroke
+			(width 0)
+			(type default)
+		)
+	)
+	(wire
+		(pts
 			(xy 130.81 128.27) (xy 81.28 128.27)
 		)
@@
 	(wire
 		(pts
-			(xy 58.42 105.41) (xy 58.42 81.28)
+			(xy 58.42 81.28) (xy 58.42 107.95)
 		)
 		(stroke
@@
 	(wire
 		(pts
-			(xy 49.53 105.41) (xy 58.42 105.41)
+			(xy 90.17 86.36) (xy 86.36 86.36)
 		)
 		(stroke
@@
 	(wire
 		(pts
+			(xy 86.36 86.36) (xy 86.36 88.9)
+		)
+		(stroke
+			(width 0)
+			(type default)
+		)
+	)
+	(wire
+		(pts
 			(xy 135.89 96.52) (xy 127 96.52)
 		)
@@
 	(wire
 		(pts
+			(xy 86.36 88.9) (xy 78.74 88.9)
+		)
+		(stroke
+			(width 0)
+			(type default)
+		)
+	)
+	(wire
+		(pts
 			(xy 34.29 62.23) (xy 34.29 69.85)
 		)
@@
 	(wire
 		(pts
+			(xy 62.23 83.82) (xy 62.23 105.41)
+		)
+		(stroke
+			(width 0)
+			(type default)
+		)
+	)
+	(wire
+		(pts
 			(xy 81.28 96.52) (xy 85.09 96.52)
 		)
@@
 	(wire
 		(pts
-			(xy 63.5 120.65) (xy 105.41 120.65)
+			(xy 63.5 120.65) (xy 78.74 120.65)
 		)
 		(stroke
@@
 	(wire
 		(pts
+			(xy 78.74 120.65) (xy 105.41 120.65)
+		)
+		(stroke
+			(width 0)
+			(type default)
+		)
+	)
+	(wire
+		(pts
 			(xy 130.81 91.44) (xy 130.81 128.27)
 		)
@@
 	(wire
 		(pts
+			(xy 62.23 105.41) (xy 49.53 105.41)
+		)
+		(stroke
+			(width 0)
+			(type default)
+		)
+	)
+	(wire
+		(pts
 			(xy 77.47 62.23) (xy 68.58 62.23)
 		)
@@
 		)
 		(stroke
-			(width 0)
-			(type default)
-		)
-	)
-	(wire
-		(pts
-			(xy 62.23 83.82) (xy 62.23 107.95)
-		)
-		(stroke
